Commit message: Restructure project: flatten src/, group assets, rename simulation.py

File: scenes/h2017/h2017.urdf (robot description, URDF)
Before this commit: robot h2017, 8 links, 7 joints
Links:
- link base_link: geometry collision mesh filename=meshes_collision/H2017_0_0.dae scale=0.001 0.001 0.001; visual mesh filename=meshes_white/H2017_0_0.dae scale=0.001 0.001 0.001
- link link_1: geometry collision mesh filename=meshes_collision/H2017_1_0.dae scale=0.001 0.001 0.001; visual mesh filename=meshes_white/H2017_1_0.dae scale=0.001 0.001 0.001
- link link_2: geometry collision mesh filename=meshes_collision/H2017_2_0.dae scale=0.001 0.001 0.001; collision mesh filename=meshes_collision/H2017_2_1.dae scale=0.001 0.001 0.001
- link link_3: geometry collision mesh filename=meshes_collision/H2017_3_0.dae scale=0.001 0.001 0.001; visual mesh filename=meshes_white/H2017_3_0.dae scale=0.001 0.001 0.001
- link link_4: geometry collision mesh filename=meshes_collision/H2017_4_0.dae scale=0.001 0.001 0.001; collision mesh filename=meshes_collision/H2017_4_1.dae scale=0.001 0.001 0.001
- link link_5: geometry collision mesh filename=meshes_collision/H2017_5_0.dae scale=0.001 0.001 0.001; visual mesh filename=meshes_white/H2017_5_0.dae scale=0.001 0.001 0.001
- link link_6: geometry collision mesh filename=meshes_collision/H2017_6_0.dae scale=0.001 0.001 0.001; visual mesh filename=meshes_white/H2017_6_0.dae scale=0.001 0.001 0.001
